File: kicad_receiver/receiver.kicad_pcb (KiCad board)
At the start: 2 copper layers, 28 parts, among them J1 Conn_01x05_Male, J2 Conn_01x01, U1 LP2985-3.3, U2 LP2985-3.3, U3 STM32F030F4Px, U4 NRF24L01_Breakout, U5 TP4056, U6 L9110, U7 MT3608

Commit message: more stuff added
Parts:
- added C13: 0.1uf, Capacitor_SMD:C_0603_1608Metric_Pad1.05x0.95mm_HandSolder, F.Cu at (196.7, 35.5)
- added C14: 10uf, Capacitor_SMD:C_0603_1608Metric_Pad1.05x0.95mm_HandSolder, F.Cu at (167.4, 63.7)
- added C15: 0.1uf, Capacitor_SMD:C_0603_1608Metric_Pad1.05x0.95mm_HandSolder, F.Cu at (178.8, 55.2)
- added C16: 22uf, Capacitor_SMD:C_0805_2012Metric_Pad1.15x1.40mm_HandSolder, F.Cu at (162.9, 63.9)
- added C17: 22uf, Capacitor_SMD:C_0805_2012Metric_Pad1.15x1.40mm_HandSolder, F.Cu at (178.0, 52.4)
- added C18: 10uf, Capacitor_SMD:C_0805_2012Metric_Pad1.15x1.40mm_HandSolder, F.Cu at (196.9, 32.7)
- added C19: 0.1uf, Capacitor_SMD:C_0603_1608Metric_Pad1.05x0.95mm_HandSolder, F.Cu at (196.7, 38.0)
- added C20: 10uf, Capacitor_SMD:C_0603_1608Metric_Pad1.05x0.95mm_HandSolder, F.Cu at (191.5, 41.8)
- added C21: 0.1uf, Capacitor_SMD:C_0603_1608Metric_Pad1.05x0.95mm_HandSolder, F.Cu at (171.8, 63.6)
- added D3: SS34, Diode_SMD:D_2114_3652Metric, F.Cu at (172.8, 57.0)
- added J3: Conn_01x01, Connector_Wire:SolderWirePad_1x01_SMD_5x10mm, F.Cu at (159.8, 55.7)
- added J4: Conn_01x01, Connector_Wire:SolderWirePad_1x01_SMD_5x10mm, F.Cu at (151.3, 58.3)
- added J5: Conn_01x01, Connector_Wire:SolderWirePad_1x01_SMD_5x10mm, F.Cu at (172.3, 37.0)
- added J6: Conn_01x01, Connector_Wire:SolderWirePad_1x01_SMD_5x10mm, F.Cu at (172.3, 48.6)
- added J7: Conn_01x01, Connector_Wire:SolderWirePad_1x01_SMD_5x10mm, F.Cu at (185.4, 37.0)
- added L1: 22uh, Inductor_SMD:L_10.4x10.4_H4.8, F.Cu at (151.0, 37.2)
- added R10: ?, Resistor_SMD:R_0603_1608Metric_Pad1.05x0.95mm_HandSolder, F.Cu at (191.2, 51.8)
- added R11: ?, Resistor_SMD:R_0603_1608Metric_Pad1.05x0.95mm_HandSolder, F.Cu at (183.2, 54.7)
- added R12: 10k, Resistor_SMD:R_0603_1608Metric_Pad1.05x0.95mm_HandSolder, F.Cu at (191.5, 46.8)
- added R13: 10k, Resistor_SMD:R_0603_1608Metric_Pad1.05x0.95mm_HandSolder, F.Cu at (186.7, 49.5)
- added R14: 220, Resistor_SMD:R_0603_1608Metric_Pad1.05x0.95mm_HandSolder, F.Cu at (195.8, 41.8)
- added R15: 220, Resistor_SMD:R_0603_1608Metric_Pad1.05x0.95mm_HandSolder, F.Cu at (186.9, 52.0)
- added R6: 10k, Resistor_SMD:R_0603_1608Metric_Pad1.05x0.95mm_HandSolder, F.Cu at (195.8, 44.3)
- added R7: 10k, Resistor_SMD:R_0603_1608Metric_Pad1.05x0.95mm_HandSolder, F.Cu at (179.8, 60.2)
- added R8: 220, Resistor_SMD:R_0603_1608Metric_Pad1.05x0.95mm_HandSolder, F.Cu at (176.1, 63.5)
- added R9: 220, Resistor_SMD:R_0603_1608Metric_Pad1.05x0.95mm_HandSolder, F.Cu at (171.8, 66.1)
- added U10: L9110, lib:L9110, F.Cu at (166.0, 53.9)
- added U11: 4N26, Package_DIP:DIP-6_W7.62mm_SMDSocket_SmallPads, F.Cu at (150.6, 47.9)
- added U12: 4N26, Package_DIP:DIP-6_W7.62mm_SMDSocket_SmallPads, F.Cu at (163.2, 35.9)
- added U8: 4N26, Package_DIP:DIP-6_W7.62mm_SMDSocket_SmallPads, F.Cu at (163.2, 45.3)
- added U9: 4N26, Package_DIP:DIP-6_W7.62mm_SMDSocket_SmallPads, F.Cu at (142.1, 57.2)
- C1, C10, C11, C12, C2, C8, C9: value 10мкф -> 10uf
- C3, C4, C7: value 0.1мкф -> 0.1uf
- C5, C6: value 0.01мкф -> 0.01uf
- R3, R4: footprint Resistor_SMD:R_0603_1608Metric_Pad1.05x0.95mm_HandSolder -> Resistor_SMD:R_0805_2012Metric_Pad1.15x1.40mm_HandSolder
- moved J2 104.0 mm to (178.9, 37.0)
- moved C5 78.5 mm to (195.8, 46.8)
- moved U1 76.6 mm to (191.6, 33.6)
- moved U3 70.4 mm to (180.1, 46.9)
- moved R1 67.2 mm to (191.5, 44.3)
- moved U2 67.2 mm to (191.6, 38.2)
- moved C3 66.4 mm to (187.5, 54.5)
- moved C11 63.6 mm to (183.2, 57.2)
- moved C6 60.8 mm to (186.7, 47.0)
- moved C12 60.7 mm to (182.5, 52.2)
- moved C8 57.2 mm to (184.1, 59.7)
- moved R4 54.3 mm to (186.9, 44.3)
- moved C2 52.2 mm to (191.1, 49.3)
- moved R5 52.0 mm to (178.8, 57.7)
- moved R2 51.4 mm to (175.4, 61.0)
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Connections:
- net tim15ch1 renamed Net-(U3-Pad8)
- net tim15ch2 renamed Net-(U3-Pad9)
- U3 pad 14: Net-(U3-Pad14) -> FB_PWM
- U3 pad 17: tim1ch2 -> FF_PWM
- U3 pad 18: tim1ch3 -> Net-(U3-Pad18)
- U4 pad 8: Net-(U4-Pad8) -> Net-(U3-Pad18)
- U5 pad 9: Net-(C11-Pad1) -> BAT-
- U6 pad 2: Net-(U6-Pad2) -> Vconv
- U6 pad 3: Net-(U6-Pad3) -> Vconv
- U6 pad 5: Net-(U6-Pad5) -> BAT-
- U6 pad 8: Net-(U6-Pad8) -> BAT-
- U7 pad 2: Net-(U7-Pad2) -> BAT-
- U7 pad 4: Net-(U7-Pad4) -> BAT+
- U7 pad 5: Net-(U7-Pad5) -> BAT+

Commit message: refactored
Parts:
- removed C20: 10uf, Capacitor_SMD:C_0603_1608Metric_Pad1.05x0.95mm_HandSolder
- removed C21: 0.1uf, Capacitor_SMD:C_0603_1608Metric_Pad1.05x0.95mm_HandSolder
- moved C18 100.4 mm to (132.4, 109.6)
- moved J5 84.5 mm to (120.8, 104.0)
- moved C5 82.0 mm to (145.6, 111.7)
- moved C19 79.3 mm to (148.3, 100.9)
- moved R14 79.2 mm to (149.3, 105.9)
- moved R13 77.1 mm to (141.3, 111.8)
- moved C13 76.8 mm to (152.0, 97.9)
- moved J2 68.2 mm to (141.8, 94.3)
- moved R6 68.1 mm to (157.0, 100.3)
- moved R10 67.0 mm to (148.3, 103.4)
- moved C9 66.9 mm to (145.6, 109.2)
- moved R4 66.8 mm to (147.5, 98.1)
- moved C2 65.9 mm to (152.7, 102.9)
- moved C8 59.5 mm to (150.0, 108.4)
- moved R2 59.2 mm to (141.3, 109.3)
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Connections:
- U11 pad 1: FF_PWM -> TURN_LEFT
- U12 pad 1: FB_PWM -> TURN_RIGHT

Commit message: place done
Parts:
- removed C16, C17: 22uf, Capacitor_SMD:C_0805_2012Metric_Pad1.15x1.40mm_HandSolder
- removed C18: 10uf, Capacitor_SMD:C_0805_2012Metric_Pad1.15x1.40mm_HandSolder
- removed D3: SS34, Diode_SMD:D_2114_3652Metric
- removed L1: 22uh, Inductor_SMD:L_10.4x10.4_H4.8
- removed R10, R11: ?, Resistor_SMD:R_0603_1608Metric_Pad1.05x0.95mm_HandSolder
- removed U7: MT3608, Package_TO_SOT_SMD:SOT-23-6_Handsoldering
- added J8: BAT+, TestPoint:TestPoint_Pad_4.0x4.0mm, F.Cu at (174.0, 81.3)
- added J9: BAT-, TestPoint:TestPoint_Pad_4.0x4.0mm, F.Cu at (173.8, 92.2)
- J2: value Conn_01x01 -> CHG+5V; footprint Connector_Wire:SolderWirePad_1x01_SMD_5x10mm -> TestPoint:TestPoint_Pad_4.0x4.0mm
- J3: value Conn_01x01 -> M1+; footprint Connector_Wire:SolderWirePad_1x01_SMD_5x10mm -> TestPoint:TestPoint_Pad_4.0x4.0mm
- J4: value Conn_01x01 -> M1-; footprint Connector_Wire:SolderWirePad_1x01_SMD_5x10mm -> TestPoint:TestPoint_Pad_4.0x4.0mm
- J5: value Conn_01x01 -> M2+; footprint Connector_Wire:SolderWirePad_1x01_SMD_5x10mm -> TestPoint:TestPoint_Pad_4.0x4.0mm
- J6: value Conn_01x01 -> M2-; footprint Connector_Wire:SolderWirePad_1x01_SMD_5x10mm -> TestPoint:TestPoint_Pad_4.0x4.0mm
- J7: value Conn_01x01 -> CHG-; footprint Connector_Wire:SolderWirePad_1x01_SMD_5x10mm -> TestPoint:TestPoint_Pad_4.0x4.0mm
- moved U5 67.1 mm to (164.2, 71.4), turned to 180 degrees
- moved D1 66.3 mm to (153.5, 69.8), turned to 180 degrees
- moved C10 52.1 mm to (168.4, 101.6), turned to 270 degrees
- moved C1 51.6 mm to (174.0, 76.1), turned to 90 degrees
- moved U4 43.6 mm to (150.0, 76.5)
- moved R6 42.5 mm to (122.0, 76.1), turned to 90 degrees
- moved J1 42.4 mm to (145.8, 102.5), turned to 90 degrees
- moved R2 40.4 mm to (157.1, 72.2), turned to 180 degrees
- moved C13 40.1 mm to (119.0, 75.1), turned to 270 degrees
- moved J2 40.0 mm to (174.0, 70.5)
- moved R12 39.1 mm to (122.0, 95.6), turned to 270 degrees
- moved R8 38.3 mm to (129.0, 68.9), turned to 270 degrees
- moved D2 36.9 mm to (153.5, 72.2), turned to 180 degrees
- moved R15 36.4 mm to (129.0, 89.0), turned to 270 degrees
- moved C2 35.5 mm to (175.8, 76.1), turned to 90 degrees
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Connections:
- net +5V renamed Net-(D1-Pad2)
- C1 pad 2: BAT- -> GND
- C10 pad 2: BAT- -> GND
- C11 pad 2: BAT- -> GND
- C12 pad 2: BAT- -> GND
- C14 pad 1: Vconv -> BAT+
- C14 pad 2: BAT- -> GND
- C15 pad 1: Vconv -> BAT+
- C15 pad 2: BAT- -> GND
- C2 pad 2: BAT- -> GND
- C3 pad 1: BAT- -> GND
- C4 pad 2: BAT- -> GND
- C5 pad 2: BAT- -> GND
- C6 pad 2: BAT- -> GND
- C7 pad 2: BAT- -> GND
- C8 pad 2: BAT- -> GND
- C9 pad 2: BAT- -> GND
- J1 pad 1: BAT- -> GND
- J7 pad 1: BAT+ -> GND
- R12 pad 1: Vconv -> BAT+
- R13 pad 1: Vconv -> BAT+
- R14 pad 2: BAT- -> GND
- R15 pad 2: BAT- -> GND
- R5 pad 2: BAT- -> GND
- R6 pad 1: Vconv -> BAT+
- R7 pad 1: Vconv -> BAT+
- R8 pad 2: BAT- -> GND
- R9 pad 2: BAT- -> GND
- U1 pad 2: BAT- -> GND
- U10 pad 2: Vconv -> BAT+
- U10 pad 3: Vconv -> BAT+
- U10 pad 5: BAT- -> GND
- U10 pad 8: BAT- -> GND
- U11 pad 4: BAT- -> GND
- U12 pad 4: BAT- -> GND
- U2 pad 2: BAT- -> GND
- U3 pad 1: Net-(U3-Pad1) -> GND
- U3 pad 10: Net-(U3-Pad10) -> TURN_RIGHT
- U3 pad 15: BAT- -> GND
- U3 pad 9: Net-(U3-Pad9) -> TURN_LEFT
- U4 pad 1: BAT- -> GND
- U4 pad 3: Net-(U3-Pad2) -> Net-(U3-Pad7)
- U4 pad 4: Net-(U3-Pad3) -> Net-(U3-Pad6)
- U4 pad 8: Net-(U3-Pad18) -> Net-(U3-Pad8)
- U5 pad 1: BAT- -> GND
- U5 pad 3: BAT- -> GND
- U5 pad 9: BAT- -> GND
- U6 pad 2: Vconv -> BAT+
- U6 pad 3: Vconv -> BAT+
- U6 pad 5: BAT- -> GND
- U6 pad 8: BAT- -> GND
- U8 pad 4: BAT- -> GND
- U9 pad 4: BAT- -> GND
Routing:
- added copper zone on F.Cu, net GND

Commit message: fixed
Parts:
- J2, J3, J4, J5, J6, J7, J8, J9: footprint TestPoint:TestPoint_Pad_4.0x4.0mm -> TestPoint:TestPoint_Pad_2.5x2.5mm
- moved U3 122.8 mm to (26.0, 83.5), turned to 180 degrees
- moved U4 106.6 mm to (47.0, 104.0), turned to 180 degrees
- moved C3 87.1 mm to (73.8, 115.6), turned to 90 degrees
- moved C5 74.0 mm to (100.4, 54.6), turned to 90 degrees
- moved U1 71.7 mm to (103.6, 59.0)
- moved C10 71.5 mm to (105.4, 67.9)
- moved C4 71.5 mm to (102.8, 68.2)
- moved C7 71.5 mm to (100.6, 68.2)
- moved C8 69.8 mm to (98.2, 68.2), turned to 270 degrees
- moved U8 67.8 mm to (75.5, 42.0), turned to 180 degrees
- moved U9 67.8 mm to (75.0, 53.8), turned to 180 degrees
- moved C13 67.4 mm to (57.2, 48.4)
- moved C19 67.4 mm to (57.2, 68.9)
- moved J3 67.4 mm to (57.2, 43.3)
- moved J4 67.4 mm to (57.2, 54.6)
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Connections:
- net Net-(U3-Pad11) renamed SPI_SCK
- net Net-(U3-Pad12) renamed SPI_MISO
- net Net-(U3-Pad13) renamed SPI_MOSI
- U3 pad 18: Net-(U3-Pad18) -> NRF_IRQ
- U3 pad 6: Net-(U3-Pad6) -> NRF_CE
- U3 pad 7: Net-(U3-Pad7) -> NRF_CSN
- U4 pad 3: Net-(U3-Pad7) -> NRF_CE
- U4 pad 4: Net-(U3-Pad6) -> NRF_CSN
- U4 pad 8: Net-(U3-Pad8) -> NRF_IRQ
Routing:
- net Net-(C11-Pad1): track 0.00 -> 43.5 mm
- net BAT+: track 0.00 -> 34.5 mm
- net GND: track 0.00 -> 18.6 mm
- net Net-(C19-Pad2): track 0.00 -> 16.3 mm
- net Net-(C13-Pad2): track 0.00 -> 16.0 mm
- net 3v3mcu: track 0.00 -> 15.7 mm
- net Net-(D1-Pad2): track 0.00 -> 12.7 mm
- net Net-(C13-Pad1): track 0.00 -> 12.6 mm
- net Net-(C19-Pad1): track 0.00 -> 12.5 mm
- net Net-(R1-Pad1): track 0.00 -> 5.98 mm
- net Net-(R6-Pad2): track 0.00 -> 5.17 mm
- net Net-(R12-Pad2): track 0.00 -> 4.54 mm
- net Net-(R2-Pad1): track 0.00 -> 4.29 mm
- net Net-(C5-Pad1): track 0.00 -> 3.55 mm
- net Net-(D2-Pad1): track 0.00 -> 3.50 mm
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- added copper zone on B.Cu, net GND
Other:
- board outline added: 60 x 50 mm

Commit message: refactored
Parts:
- removed C19: 0.1uf, Capacitor_SMD:C_0603_1608Metric_Pad1.05x0.95mm_HandSolder
- removed the C2 at (182.9, 97.0)
- removed the C7 at (100.6, 68.2)
- removed the J2 at (185.5, 76.5)
- removed the R12 at (60.2, 69.0)
- removed R15: 220, Resistor_SMD:R_0603_1608Metric_Pad1.05x0.95mm_HandSolder
- removed U12: 4N26, Package_DIP:DIP-6_W7.62mm_SMDSocket_SmallPads
- added C10: 10uf, Capacitor_SMD:C_0805_2012Metric_Pad1.15x1.40mm_HandSolder, F.Cu at (161.7, 107.8)
- added C16: 10uf, Capacitor_SMD:C_0805_2012Metric_Pad1.15x1.40mm_HandSolder, F.Cu at (182.9, 96.8)
- added C3: 0.1uf, Capacitor_SMD:C_0805_2012Metric_Pad1.15x1.40mm_HandSolder, F.Cu at (118.5, 142.0)
- added J6: CHG+5V, TestPoint:TestPoint_Pad_2.5x2.5mm, F.Cu at (183.0, 80.0)
- added R10: 220, Resistor_SMD:R_0603_1608Metric_Pad1.05x0.95mm_HandSolder, F.Cu at (155.5, 87.6)
- added R5: 10k, Resistor_SMD:R_0603_1608Metric_Pad1.05x0.95mm_HandSolder, F.Cu at (140.6, 79.8)
- added U10: 4N26, Package_DIP:DIP-6_W7.62mm_SMDSocket_SmallPads, F.Cu at (149.8, 106.2)
- C1, C8: footprint Capacitor_SMD:C_0603_1608Metric_Pad1.05x0.95mm_HandSolder -> Capacitor_SMD:C_0805_2012Metric_Pad1.15x1.40mm_HandSolder
- C11, C12, C14: value 10uf -> 0.1uf; footprint Capacitor_SMD:C_0603_1608Metric_Pad1.05x0.95mm_HandSolder -> Capacitor_SMD:C_0805_2012Metric_Pad1.15x1.40mm_HandSolder
- C13, C15: value 0.1uf -> 10uf; footprint Capacitor_SMD:C_0603_1608Metric_Pad1.05x0.95mm_HandSolder -> Capacitor_SMD:C_0805_2012Metric_Pad1.15x1.40mm_HandSolder
- C4: value 0.1uf -> 0.01uf; footprint Capacitor_SMD:C_0603_1608Metric_Pad1.05x0.95mm_HandSolder -> Capacitor_SMD:C_0805_2012Metric_Pad1.15x1.40mm_HandSolder
- C5: value 0.01uf -> 0.1uf; footprint Capacitor_SMD:C_0603_1608Metric_Pad1.05x0.95mm_HandSolder -> Capacitor_SMD:C_0805_2012Metric_Pad1.15x1.40mm_HandSolder
- C6: value 0.01uf -> 10uf; footprint Capacitor_SMD:C_0603_1608Metric_Pad1.05x0.95mm_HandSolder -> Capacitor_SMD:C_0805_2012Metric_Pad1.15x1.40mm_HandSolder
- C9: value 10uf -> 0.01uf; footprint Capacitor_SMD:C_0603_1608Metric_Pad1.05x0.95mm_HandSolder -> Capacitor_SMD:C_0805_2012Metric_Pad1.15x1.40mm_HandSolder
- R13: value 10k -> 220
- R8: value 220 -> 10k
- moved C13 137.6 mm to (182.9, 104.3), turned to 0 degrees
- moved U2 132.3 mm to (142.5, 146.2)
- moved U3 123.7 mm to (170.0, 116.8), turned to 270 degrees
- moved R8 107.4 mm to (140.4, 121.0), turned to 0 degrees
- moved R13 102.5 mm to (156.0, 121.9), turned to 270 degrees
- moved R6 101.7 mm to (140.4, 112.0), turned to 0 degrees
- moved R11 95.4 mm to (155.8, 99.9), turned to 270 degrees
- moved R12 89.8 mm to (155.8, 112.4), turned to 270 degrees
- moved U6 89.6 mm to (140.5, 116.3), turned to 270 degrees
- moved C5 88.8 mm to (114.8, 142.3), turned to 270 degrees
- moved J4 88.5 mm to (130.8, 112.5)
- moved C8 88.2 mm to (182.9, 92.8), turned to 0 degrees
- moved J5 86.6 mm to (130.8, 120.0)
- moved U9 84.6 mm to (149.8, 93.5), turned to 90 degrees
- moved C6 84.6 mm to (177.2, 103.3), turned to 270 degrees
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- renumbered C3 to C2, C10 to C7, J3 to J2, J4 to J3, J5 to J4, J6 to J5, R9 to R11, R14 to R12, R3 to R2, R4 to R3, R2 to R4, R5 to R9, U3 to U2, U4 to U3, U2 to U4, U6 to U5, U10 to U6, U5 to U7
Connections:
- C11 pad 2: GND -> Net-(C11-Pad2)
- C12 pad 1: BAT+ -> Net-(C12-Pad1)
- C12 pad 2: GND -> Net-(C12-Pad2)
- C13 pad 1: Net-(C13-Pad1) -> BAT+
- C13 pad 2: Net-(C13-Pad2) -> GND
- C15 pad 1: BAT+ -> Net-(C15-Pad1)
- C4 pad 1: 3v3mcu -> Net-(C4-Pad1)
- C5 pad 1: Net-(C5-Pad1) -> 3v3mcu
- C6 pad 1: Net-(C6-Pad1) -> 3v3mcu
- C8 pad 1: 3v3mcu -> BAT+
- C9 pad 1: 3v3radio -> Net-(C9-Pad1)
- J2 pad 1: Net-(C13-Pad1) -> Net-(C11-Pad1)
- J3 pad 1: Net-(C13-Pad2) -> Net-(C11-Pad2)
- J4 pad 1: Net-(C19-Pad1) -> Net-(C12-Pad1)
- J5 pad 1: Net-(C19-Pad2) -> Net-(C12-Pad2)
- R12 pad 1: Net-(R14-Pad1) -> Net-(R12-Pad1)
- R13 pad 1: BAT+ -> Net-(R13-Pad1)
- R13 pad 2: Net-(R13-Pad2) -> GND
- R2 pad 2: Net-(C11-Pad1) -> Net-(C15-Pad1)
- R3 pad 2: Net-(C11-Pad1) -> Net-(C15-Pad1)
- R8 pad 1: Net-(R8-Pad1) -> BAT+
- R8 pad 2: GND -> Net-(R8-Pad2)
- U1 pad 4: Net-(C5-Pad1) -> Net-(C4-Pad1)
- U11 pad 1: TURN_LEFT -> TURN_RIGHT
- U11 pad 2: Net-(R14-Pad1) -> Net-(R13-Pad1)
- U11 pad 5: Net-(R12-Pad2) -> Net-(R8-Pad2)
- U4 pad 4: Net-(C6-Pad1) -> Net-(C9-Pad1)
- U5 pad 1: Net-(C13-Pad1) -> Net-(C11-Pad1)
- U5 pad 4: Net-(C13-Pad2) -> Net-(C11-Pad2)
- U5 pad 7: Net-(R6-Pad2) -> Net-(R5-Pad2)
- U6 pad 1: Net-(C19-Pad1) -> Net-(C12-Pad1)
- U6 pad 4: Net-(C19-Pad2) -> Net-(C12-Pad2)
- U6 pad 6: Net-(R13-Pad2) -> Net-(R8-Pad2)
- U6 pad 7: Net-(R12-Pad2) -> Net-(R6-Pad2)
- U7 pad 4: Net-(C11-Pad1) -> Net-(C15-Pad1)
- U7 pad 8: Net-(C11-Pad1) -> Net-(C15-Pad1)
- U8 pad 2: Net-(R8-Pad1) -> Net-(R10-Pad1)
- U8 pad 5: Net-(R6-Pad2) -> Net-(R5-Pad2)
Routing:
- net BAT+: track 34.5 -> 159.6 mm, vias 0 -> 20
- net Net-(C15-Pad1): track 0.00 -> 43.5 mm
- net Net-(C11-Pad1): track 43.5 -> 11.8 mm
- net Net-(C19-Pad2): track 16.3 -> 0.00 mm
- net Net-(C13-Pad2): track 16.0 -> 0.00 mm
- net 3v3mcu: track 15.7 -> 0.00 mm
- net Net-(R7-Pad2): track 0.00 -> 15.1 mm
- net Net-(C12-Pad1): track 0.00 -> 14.0 mm
- net Net-(R5-Pad2): track 0.00 -> 13.7 mm
- net Net-(C12-Pad2): track 0.00 -> 13.7 mm
- net Net-(R8-Pad2): track 0.00 -> 13.1 mm
- net Net-(R6-Pad2): track 5.17 -> 17.8 mm
- net Net-(C13-Pad1): track 12.6 -> 0.00 mm
- net Net-(C19-Pad1): track 12.5 -> 0.00 mm
- net Net-(C11-Pad2): track 0.00 -> 11.9 mm
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
Commit message: almost routed
Parts:
- moved C5 63.5 mm to (166.7, 105.8), turned to 180 degrees
- moved C3 62.7 mm to (166.7, 102.0), turned to 180 degrees
- moved C7 60.3 mm to (166.2, 98.5), turned to 180 degrees
- moved C2 56.9 mm to (179.2, 111.4)
- moved U2 55.3 mm to (175.2, 101.8), turned to 90 degrees
- moved J1 35.2 mm to (166.2, 109.5), turned to 90 degrees
- moved C9 15.2 mm to (159.0, 88.2), turned to 90 degrees
- moved C4 14.5 mm to (168.2, 93.5), turned to 270 degrees
- moved C10 14.5 mm to (159.0, 93.5), turned to 90 degrees
- moved C6 11.2 mm to (171.8, 93.5), turned to 90 degrees
- moved U1 10.4 mm to (176.3, 93.5), turned to 180 degrees
- moved U4 9.95 mm to (163.4, 93.5)
- moved U3 0.75 mm to (170.0, 117.5)
Routing:
- net BAT+: track 159.6 -> 205.9 mm
- net 3v3mcu: track 0.00 -> 36.2 mm
- net 3v3radio: track 9.67 -> 22.9 mm
- net Net-(C4-Pad1): track 0.00 -> 9.37 mm
- net GND: track 9.62 -> 17.7 mm, vias 30 -> 39
- net FB_PWM: track 0.00 -> 7.44 mm, vias 0 -> 2
- net FF_PWM: track 0.00 -> 6.92 mm, vias 0 -> 2
- net RST: track 0.00 -> 5.42 mm, vias 0 -> 1
- net TURN_LEFT: track 0.00 -> 5.03 mm, vias 0 -> 2
- net TURN_RIGHT: track 0.00 -> 4.84 mm, vias 0 -> 2
- net SPI_SCK: track 3.08 -> 5.65 mm, vias 1 -> 2
- net NRF_CSN: track 3.11 -> 5.28 mm, vias 1 -> 2
- net SPI_MISO: track 3.00 -> 5.15 mm, vias 1 -> 2
- net NRF_IRQ: track 2.97 -> 5.07 mm, vias 1 -> 2
- net SWCLK: track 0.00 -> 2.08 mm, vias 0 -> 1
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
Commit message: done!
Parts:
- moved C2 17.7 mm to (161.6, 109.5), turned to 0 degrees
- moved J1 10.3 mm to (166.5, 99.2), turned to 0 degrees
- moved C3 5.02 mm to (161.7, 102.5)
- moved C5 5.02 mm to (161.7, 106.2)
- moved C7 5.02 mm to (161.2, 99.0)
- moved U2 3.61 mm to (173.2, 104.8)
- moved U3 1.00 mm to (170.0, 118.5)
Connections:
- J1 pad 1: GND -> 3v3mcu
- J1 pad 2: 3v3mcu -> SWCLK
- J1 pad 4: SWCLK -> GND
- U2 pad 18: NRF_IRQ -> Net-(U2-Pad18)
- U2 pad 8: Net-(U2-Pad8) -> NRF_IRQ
Routing:
- net FB_PWM: track 7.44 -> 48.3 mm
- net FF_PWM: track 6.92 -> 44.0 mm
- net TURN_RIGHT: track 4.84 -> 39.0 mm
- net SPI_MOSI: track 5.04 -> 35.5 mm, vias 2 -> 0
- net TURN_LEFT: track 5.03 -> 35.4 mm
- net NRF_IRQ: track 5.07 -> 31.5 mm
- net SPI_MISO: track 5.15 -> 29.7 mm
- net SPI_SCK: track 5.65 -> 28.0 mm, vias 2 -> 0
- net NRF_CSN: track 5.28 -> 17.8 mm, vias 2 -> 0
- net NRF_CE: track 5.17 -> 16.5 mm, vias 2 -> 0
- net RST: track 5.42 -> 12.1 mm, vias 1 -> 0
- net SWIO: track 1.96 -> 6.74 mm, vias 1 -> 0
- net BAT+: track 205.9 -> 209.6 mm
- net Net-(C11-Pad1): track 11.8 -> 14.1 mm
- net Net-(C11-Pad2): track 11.9 -> 14.1 mm
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
Commit message: refactored
Routing:
- net BAT+: track 209.6 -> 232.0 mm
- net GND: vias 39 -> 35
